File: hw/catfeeder.sch (KiCad schematic (older format))
At the start: 15 parts, among them IC1 ATMEGA328-P, P1 LCD, P2 PROG, P3 SERVO, P4 3_3_SUP, P5 ROT_SWITCH, P6 CONN_01X06, P7 BUTTON, P8 HC-SR04, P9 WS2812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

Commit message: Update catfeeder schematics
Connections:
- net RESET: now also U2.4 (GPIO2)
Changed lines of the file:
@@
 L GND #PWR010
 U 1 1 5765AD23
-P 5700 6500
-F 0 "#PWR010" H 5700 6250 50  0001 C CNN
-F 1 "GND" H 5705 6327 50  0000 C CNN
-F 2 "" H 5700 6500 50  0000 C CNN
-F 3 "" H 5700 6500 50  0000 C CNN
-	1    5700 6500
+P 5850 6150
+F 0 "#PWR010" H 5850 5900 50  0001 C CNN
+F 1 "GND" H 5855 5977 50  0000 C CNN
+F 2 "" H 5850 6150 50  0000 C CNN
+F 3 "" H 5850 6150 50  0000 C CNN
+	1    5850 6150
 	1    0    0    -1
 $EndComp
@@
 	10250 1250 10350 1250
 Wire Wire Line
-	5700 6500 5500 6500
-Wire Wire Line
 	3150 4050 3650 4050
 Wire Wire Line
@@
 	1    0    0    -1
 $EndComp
+Text Label 5900 6600 0    60   ~ 0
+RESET
+Wire Wire Line
+	5500 6500 5500 6100
+Wire Wire Line
+	5500 6100 5850 6100
+Wire Wire Line
+	5850 6100 5850 6150
+Wire Wire Line
+	5500 6600 5900 6600
 $EndSCHEMATC
