File: hw/catfeeder_v2.sch (KiCad schematic (older format))
At the start: 13 parts, among them J1 Conn_01x02, J2 Conn_01x02, J3 Conn_01x02, J4 Conn_01x04, J5 CONN_SENSOR, J6 CONN_ENC, J7 CONN_CLK, U1 NodeMCU_1.0_(ESP-12E), U2 PCF8574

Commit message: Use submodule for esp footprint
Parts:
- removed J1, J2, J3: Conn_01x02, symbol Conn_01x02
- removed J5: CONN_SENSOR, symbol Conn_01x04
- removed J6: CONN_ENC, symbol Conn_01x05
- removed J7: CONN_CLK, symbol Conn_01x06
- removed R1, R2, R3: R, symbol R
- removed U2: PCF8574, symbol PCF8574
- added DRV2: POLOLU-DRV8825, POLOLU-DRV8825:POLOLU-DRV8825, symbol pololu-drv8825:POLOLU-DRV8825
- added J1: CONN_BEEPER, Connector_PinHeader_2.54mm:PinHeader_1x02_P2.54mm_Vertical, symbol catfeeder_v2-rescue:Conn_01x02
- added J11: CONN_MOT2, Connector_PinHeader_2.54mm:PinHeader_1x04_P2.54mm_Vertical, symbol catfeeder_v2-rescue:Conn_01x04
- added J2: CONN_SENSOR_ADC, Connector_PinHeader_2.54mm:PinHeader_1x03_P2.54mm_Vertical, symbol Connector_Generic:Conn_01x03
- added J3: CONN_SENSOR, Connector_PinHeader_2.54mm:PinHeader_1x03_P2.54mm_Vertical, symbol Connector_Generic:Conn_01x03
- added J6: CONN_LCD, Connector_IDC:IDC-Header_2x05_P2.54mm_Vertical, symbol Connector_Generic:Conn_02x05_Odd_Even
- added J8: CONN_POWER, TerminalBlock:TerminalBlock_bornier-2_P5.08mm, symbol catfeeder_v2-rescue:Conn_01x02
- added JP1, JP2, JP3, JP4, JP5, JP6: Jumper, Resistor_SMD:R_0805_2012Metric_Pad1.15x1.40mm_HandSolder, symbol Device:Jumper
- added Q1: IRLML6402, Package_TO_SOT_SMD:SOT-23, symbol Transistor_FET:IRLML6402
- added R1, R2: R, Resistor_THT:R_Axial_DIN0207_L6.3mm_D2.5mm_P10.16mm_Horizontal, symbol catfeeder_v2-rescue:R
- added U2: LM317_3PinPackage, Package_TO_SOT_THT:TO-220-3_Vertical, symbol Regulator_Linear:LM317_3PinPackage
- DRV1: footprint (none) -> POLOLU-DRV8825:POLOLU-DRV8825; symbol POLOLU-DRV8825 -> pololu-drv8825:POLOLU-DRV8825
- J4: value Conn_01x04 -> CONN_MOT1; footprint (none) -> Connector_PinHeader_2.54mm:PinHeader_1x04_P2.54mm_Vertical; symbol Conn_01x04 -> catfeeder_v2-rescue:Conn_01x04
- U1: footprint (none) -> ESP8266:ESP12F-Devkit-V3; symbol NodeMCU_1.0_(ESP-12E) -> ESP8266:NodeMCU_1.0_(ESP-12E)
Connections:
- net labels added: BEEPER, LCD_INT, MOT10, MOT11, MOT12, MOT1_DIR, MOT1_STEP, MOT20, MOT21, MOT22, MOT2_DIR, MOT2_STEP, SENSOR_ANALOG_IN, VCC
- net labels removed: ENC_ROT1, ENC_ROT2, ENC_SW, LCD_D4, LCD_D5, LCD_D6, LCD_D7, LCD_EN, LCD_RS, LCD_RW, MOT0, MOT1, MOT2, MOT_DIR, MOT_STEP, SENSOR_OUT
- wire segments 65 -> 111
- no-connect marks 4 -> 6
Other:
- moved on the sheet: J4

Commit message: hw: Add missing pullup resistors for I2C
Parts:
- added R3, R4, R5: R, Resistor_THT:R_Axial_DIN0207_L6.3mm_D2.5mm_P10.16mm_Horizontal, symbol catfeeder_v2-rescue:R
- J1: footprint Connector_PinHeader_2.54mm:PinHeader_1x02_P2.54mm_Vertical -> Connector_JST:JST_XH_B02B-XH-A_1x02_P2.50mm_Vertical
- J11, J4: footprint Connector_PinHeader_2.54mm:PinHeader_1x04_P2.54mm_Vertical -> Connector_JST:JST_XH_B04B-XH-A_1x04_P2.50mm_Vertical
- J2, J3: footprint Connector_PinHeader_2.54mm:PinHeader_1x03_P2.54mm_Vertical -> Connector_JST:JST_XH_B03B-XH-A_1x03_P2.50mm_Vertical
- R1, R2: footprint Resistor_THT:R_Axial_DIN0207_L6.3mm_D2.5mm_P10.16mm_Horizontal -> Resistor_SMD:R_0805_2012Metric_Pad1.15x1.40mm_HandSolder
Connections:
- net +3V3: now also R3.1, R4.1, R5.2
- net I2C_SCL: now also R4.2
- net I2C_SDA: now also R3.2
- net LCD_INT: now also R5.1
- net SENSOR_1: now reaches U1.4 (SD3(GPIO10))
- net SENSOR_1: now also J3.3 (Pin_3)
- net MOT_ENABLE: now reaches DRV1.1 (ENABLE)
- net MOT_ENABLE: now also DRV2.1 (ENABLE), U1.22 (D6(GPIO12))
- removed net SENSOR_IN: J3.3 (Pin_3), U1.22 (D6(GPIO12))
- no-connect marks 6 -> 16

Commit message: Move INTPIN to GPIO3
Parts:
- removed R5: R, Resistor_THT:R_Axial_DIN0207_L6.3mm_D2.5mm_P10.16mm_Horizontal, symbol catfeeder_v2-rescue:R
Connections:
- net LCD_INT: now also U1.19 (RX(DPIO3)); no longer U1.27 (D3(GPIO0))
Changed lines of the file:
@@
 Wire Wire Line
 	2650 4300 2200 4300
-Wire Wire Line
-	4200 6100 3950 6100
 Text Label 4300 6200 0    60   ~ 0
 MOT2_STEP
@@
 Text Label 4000 4400 0    60   ~ 0
 LCD_INT
-Text Label 4200 6100 0    60   ~ 0
+Text Label 4200 6900 0    60   ~ 0
 LCD_INT
 $Comp
@@
 Text Label 4200 6600 0    60   ~ 0
 MOT_ENABLE
-Wire Wire Line
-	4000 4400 3850 4400
-$Comp
-L catfeeder_v2-rescue:R R5
-U 1 1 5D63CAC2
-P 3850 4550
-F 0 "R5" H 3920 4596 50  0000 L CNN
-F 1 "R" H 3920 4505 50  0000 L CNN
-F 2 "Resistor_THT:R_Axial_DIN0207_L6.3mm_D2.5mm_P10.16mm_Horizontal" V 3780 4550 50  0001 C CNN
-F 3 "" H 3850 4550 50  0001 C CNN
-	1    3850 4550
-	1    0    0    -1
-$EndComp
-Connection ~ 3850 4400
-Wire Wire Line
-	3850 4400 3150 4400
-Wire Wire Line
-	3850 4700 4450 4700
-Wire Wire Line
-	4450 4700 4450 4200
 $Comp
 L catfeeder_v2-rescue:R R3
@@
 F 3 "" H 3850 4000 50  0001 C CNN
 	1    3850 4000
-	1    0    0    -1
-$EndComp
-$Comp
-L power:+3.3V #PWR010
-U 1 1 5D65AC1F
-P 4450 4200
-F 0 "#PWR010" H 4450 4050 50  0001 C CNN
-F 1 "+3.3V" H 4465 4373 50  0000 C CNN
-F 2 "" H 4450 4200 50  0001 C CNN
-F 3 "" H 4450 4200 50  0001 C CNN
-	1    4450 4200
 	1    0    0    -1
 $EndComp
@@
 NoConn ~ 2350 7000
 NoConn ~ 3950 7000
-NoConn ~ 3950 6900
 NoConn ~ 9100 -900
+Wire Wire Line
+	3950 6900 4200 6900
+NoConn ~ 3950 6100
+Wire Wire Line
+	3150 4400 4000 4400
 $EndSCHEMATC
